File: circuits/lia_robot/lia_robot.kicad_sch (KiCad schematic)
At the start: 13 parts, among them J1 Jack-DC, J2 IR_SENSORS, J3 L298N, SW1 SW_DIP_x01, SW2 SW_Push_Dual, SW3 SW_Push_Dual, SW4 SW_Push_Dual, U1 AMS1117, U2 ESP32-DEVKIT-V1

Commit message: feat: adding mechanical assets
Other:
- note added: "Botão 2"
- note added: "Botão1"
- note added: "Botão3"
- moved on the sheet: J3
Changed lines of the file:
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@@
     (stroke (width 0) (type default) (color 0 0 0 0))
   )
-  (wire (pts (xy 123.19 110.49) (xy 129.54 110.49))
+  (wire (pts (xy 129.54 110.49) (xy 135.89 110.49))
     (stroke (width 0) (type default) (color 0 0 0 0))
   )
@@
     (stroke (width 0) (type default) (color 0 0 0 0))
   )
-  (wire (pts (xy 123.19 113.03) (xy 129.54 113.03))
+  (wire (pts (xy 129.54 113.03) (xy 135.89 113.03))
     (stroke (width 0) (type default) (color 0 0 0 0))
   )
@@
     (stroke (width 0) (type default) (color 0 0 0 0))
   )
-  (wire (pts (xy 123.19 115.57) (xy 129.54 115.57))
+  (wire (pts (xy 129.54 115.57) (xy 135.89 115.57))
     (stroke (width 0) (type default) (color 0 0 0 0))
   )
@@
     (stroke (width 0) (type default) (color 0 0 0 0))
   )
-  (wire (pts (xy 123.19 120.65) (xy 129.54 120.65))
+  (wire (pts (xy 129.54 120.65) (xy 135.89 120.65))
     (stroke (width 0) (type default) (color 0 0 0 0))
   )
@@
     (stroke (width 0) (type default) (color 0 0 0 0))
   )
-  (wire (pts (xy 123.19 118.11) (xy 129.54 118.11))
+  (wire (pts (xy 129.54 118.11) (xy 135.89 118.11))
     (stroke (width 0) (type default) (color 0 0 0 0))
   )
@@
     (stroke (width 0) (type default) (color 0 0 0 0))
   )
-  (wire (pts (xy 123.19 123.19) (xy 129.54 123.19))
+  (wire (pts (xy 129.54 123.19) (xy 135.89 123.19))
     (stroke (width 0) (type default) (color 0 0 0 0))
   )
@@
     (effects (font (size 1.27 1.27)) (justify left bottom))
   )
-  (label "IN1" (at 125.73 113.03 0)
+  (text "Botão1\n" (at 24.13 58.42 0)
+    (effects (font (size 1.27 1.27)) (justify left bottom))
+  )
+  (text "Botão3\n" (at 24.13 101.6 0)
+    (effects (font (size 1.27 1.27)) (justify left bottom))
+  )
+  (text "Botão 2\n" (at 24.13 77.47 0)
+    (effects (font (size 1.27 1.27)) (justify left bottom))
+  )
+  (label "IN1" (at 132.08 113.03 0)
     (effects (font (size 1.27 1.27)) (justify left bottom))
   )
@@
     (effects (font (size 1.27 1.27)) (justify left bottom))
   )
-  (label "ENA" (at 125.73 110.49 0)
+  (label "ENA" (at 132.08 110.49 0)
     (effects (font (size 1.27 1.27)) (justify left bottom))
   )
@@
     (effects (font (size 1.27 1.27)) (justify left bottom))
   )
-  (label "ENB" (at 125.73 123.19 0)
+  (label "ENB" (at 132.08 123.19 0)
     (effects (font (size 1.27 1.27)) (justify left bottom))
   )
@@
     (effects (font (size 1.27 1.27)) (justify left bottom))
   )
-  (label "IN4" (at 125.73 120.65 0)
+  (label "IN4" (at 132.08 120.65 0)
     (effects (font (size 1.27 1.27)) (justify left bottom))
   )
@@
     (effects (font (size 1.27 1.27)) (justify left bottom))
   )
-  (label "IN2" (at 125.73 115.57 0)
+  (label "IN2" (at 132.08 115.57 0)
     (effects (font (size 1.27 1.27)) (justify left bottom))
   )
@@
     (effects (font (size 1.27 1.27)) (justify left bottom))
   )
-  (label "IN3" (at 125.73 118.11 0)
+  (label "IN3" (at 132.08 118.11 0)
     (effects (font (size 1.27 1.27)) (justify left bottom))
   )
@@
     (pin "2")
   )
-  (symbol (lib_id "Connector:Conn_01x06_Male") (at 118.11 115.57 0) (unit 1)
-    (in_bom yes) (on_board yes) (fields_autoplaced)
-    (property "Reference" "J3" (id 0) (at 118.745 105.41 0))
-    (property "Value" "L298N" (id 1) (at 118.745 107.95 0))
-    (property "Footprint" "" (id 2) (at 118.11 115.57 0)
-      (effects (font (size 1.27 1.27)) hide)
-    )
-    (property "Datasheet" "~" (id 3) (at 118.11 115.57 0)
-      (effects (font (size 1.27 1.27)) hide)
-    )
+  (symbol (lib_id "Connector:Conn_01x06_Male") (at 124.46 115.57 0) (unit 1)
+    (in_bom yes) (on_board yes) (fields_autoplaced)
+    (property "Reference" "J3" (id 0) (at 125.095 105.41 0))
+    (property "Value" "L298N" (id 1) (at 125.095 107.95 0))
+    (property "Footprint" "" (id 2) (at 124.46 115.57 0)
+      (effects (font (size 1.27 1.27)) hide)
+    )
+    (property "Datasheet" "~" (id 3) (at 124.46 115.57 0)
+      (effects (font (size 1.27 1.27)) hide)
+    )
